File: hardware/tpmsniffer.kicad_pcb (KiCad board)
At the start: 2 copper layers, 25.4 x 70.4 mm, 12 parts, among them J1 Conn_01x06_Pin, U1 Pico

Commit message: Modified silkscreen
Other:
- board text added: "Aaron Kelly TPM Sniffer LAB USE ONLY"
- board text added: "https://github.com/kelemvor4/pico-tpmsniffer"
- board text removed: "hextree.io"
- board text removed: "stacksmashing"
